File: robotica/robotica.kicad_pcb (KiCad board)
At the start: 2 copper layers, 92.1 x 101 mm, 52 parts, among them J1 IZQUIERDA, J10 Conn_01x03, J11 Conn_01x03, J12 LCD, J13 LCD, J14 12V, J15 POWER, J16 Conn_01x04, J17 salidas, J18 Conn_01x05, J19 Conn_01x03, J2 DERECHA, J20 Conn_01x15, J21 Conn_01x01, J22 Conn_01x01, J23 Conn_01x04, J24 Conn_01x05, J25 Conn_01x03, J26 Conn_01x15, J27 Conn_01x01, J28 Conn_01x01, J3 salidas, J4 MOTOR, J5 MOTOR, J6 12V, J7 driv, J8 Conn_01x03, J9 Conn_01x03, K1 FINDER-36.11, K2 FINDER-36.11, Q1 2N3904, Q2 2N3904, U2 LM7805_TO220, U3 4N35, U4 4N35

Commit message: termincacion del pcb de robotica
Parts:
- added J29: Conn_01x04, Connector_PinSocket_2.54mm:PinSocket_1x04_P2.54mm_Vertical, F.Cu at (57.2, 86.2)
- added J30: Conn_01x04, Connector_PinSocket_2.54mm:PinSocket_1x04_P2.54mm_Vertical, F.Cu at (61.8, 86.2)
- added J31: Conn_01x04, Connector_PinSocket_2.54mm:PinSocket_1x04_P2.54mm_Vertical, F.Cu at (66.4, 86.2)
- moved J6 4.21 mm to (61.8, 142.7)
Routing:
- net +12V: track 138.9 -> 186.7 mm
- net +5VA: track 108.6 -> 150.8 mm
- net Net-(J17-Pin_2): track 22.7 -> 45.4 mm
- net Net-(J3-Pin_2): track 22.7 -> 45.4 mm
- net Net-(J17-Pin_3): track 8.86 -> 17.7 mm
- net Net-(J3-Pin_1): track 8.86 -> 17.7 mm
- net Net-(J3-Pin_3): track 8.86 -> 17.7 mm
- net Net-(J17-Pin_1): track 8.86 -> 17.7 mm
Other:
- board text added: "5V"
