File: robotica/robotica.kicad_sch (KiCad schematic)
At the start: 0 parts

Commit message: PCB YA REALIZADO
Parts:
- added J16: Conn_01x04, Connector_PinHeader_2.54mm:PinHeader_1x04_P2.54mm_Vertical, symbol Connector_Generic:Conn_01x04
- added J18: Conn_01x05, Connector_PinHeader_2.54mm:PinHeader_1x05_P2.54mm_Vertical, symbol Connector_Generic:Conn_01x05
- added J19: Conn_01x03, Connector_PinHeader_2.54mm:PinHeader_1x03_P2.54mm_Vertical, symbol Connector_Generic:Conn_01x03
- added J20: Conn_01x15, Connector_PinHeader_2.54mm:PinHeader_1x15_P2.54mm_Vertical, symbol Connector_Generic:Conn_01x15
- added J21, J28: Conn_01x01, Connector_PinHeader_2.54mm:PinHeader_1x01_P2.54mm_Vertical, symbol Connector_Generic:Conn_01x01
- added J22, J27: Conn_01x01, Connector_PinSocket_2.54mm:PinSocket_1x01_P2.54mm_Vertical, symbol Connector_Generic:Conn_01x01
- added J23: Conn_01x04, Connector_PinSocket_2.54mm:PinSocket_1x04_P2.54mm_Vertical, symbol Connector_Generic:Conn_01x04
- added J24: Conn_01x05, Connector_PinSocket_2.54mm:PinSocket_1x05_P2.54mm_Vertical, symbol Connector_Generic:Conn_01x05
- added J25: Conn_01x03, Connector_PinSocket_2.54mm:PinSocket_1x03_P2.54mm_Vertical, symbol Connector_Generic:Conn_01x03
- added J26: Conn_01x15, Connector_PinSocket_2.54mm:PinSocket_1x15_P2.54mm_Vertical, symbol Connector_Generic:Conn_01x15
Connections:
- net micro/GPIO0: now also J21.1 (Pin_1), J22.1 (Pin_1)
- net micro/GPIO11: now also J27.1 (Pin_1), J28.1 (Pin_1)
- net micro/GPIO13: now also J18.5 (Pin_5), J24.5 (Pin_5)
- net micro/GPIO14: now also J18.4 (Pin_4), J24.4 (Pin_4)
- net micro/GPIO15: now also J18.3 (Pin_3), J24.3 (Pin_3)
- net micro/GPIO16: now also J18.2 (Pin_2), J24.2 (Pin_2)
- net micro/GPIO17: now also J18.1 (Pin_1), J24.1 (Pin_1)
- net micro/GPIO18: now also J20.15 (Pin_15), J26.15 (Pin_15)
- net micro/GPIO19: now also J20.14 (Pin_14), J26.14 (Pin_14)
- net micro/GPIO20: now also J20.13 (Pin_13), J26.13 (Pin_13)
- net micro/GPIO21: now also J20.12 (Pin_12), J26.12 (Pin_12)
- net micro/GPIO26: now also J20.11 (Pin_11), J26.11 (Pin_11)
- net micro/GPIO33: now also J20.10 (Pin_10), J26.10 (Pin_10)
- net micro/GPIO34: now also J20.9 (Pin_9), J26.9 (Pin_9)
- net micro/GPIO35: now also J20.8 (Pin_8), J26.8 (Pin_8)
- net micro/GPIO36: now also J20.7 (Pin_7), J26.7 (Pin_7)
- net micro/GPIO37: now also J20.6 (Pin_6), J26.6 (Pin_6)
- net micro/GPIO38: now also J20.5 (Pin_5), J26.5 (Pin_5)
- net micro/GPIO39: now also J20.4 (Pin_4), J26.4 (Pin_4)
- net micro/GPIO40: now also J20.3 (Pin_3), J26.3 (Pin_3)
- net micro/GPIO41: now also J20.2 (Pin_2), J26.2 (Pin_2)
- net micro/GPIO42: now also J20.1 (Pin_1), J26.1 (Pin_1)
- net micro/GPIO45: now also J19.3 (Pin_3), J25.3 (Pin_3)
- net micro/GPIO46: now also J19.2 (Pin_2), J25.2 (Pin_2)
- net micro/GPIO6: now also J16.4 (Pin_4), J23.4 (Pin_4)
- net micro/GPIO7: now also J16.3 (Pin_3), J23.3 (Pin_3)
- net micro/GPIO8: now also J16.2 (Pin_2), J23.2 (Pin_2)
- net micro/GPIO9: now also J16.1 (Pin_1), J23.1 (Pin_1)
- net micro/RST: now also J19.1 (Pin_1), J25.1 (Pin_1)
