File: mod. de exp. FPGA spartan 6 mimasV2 - copia/DIP_SWICTH.kicad_sch (KiCad schematic)
At the start: 9 parts, among them SW1 SW_DIP_x08

Commit message: absolutamente todo
Connections:
- net 1P9: now also R8.2, SW1.9; no longer R7.2, SW1.10
- net 2P9: now also R7.2, SW1.10; no longer R8.2, SW1.9
- net 3P9: now also R6.2, SW1.11; no longer R5.2, SW1.12
- net 4P9: now also R5.2, SW1.12; no longer R6.2, SW1.11
- net 5P9: now also R4.2, SW1.13; no longer R3.2, SW1.14
- net 6P9: now also R3.2, SW1.14; no longer R4.2, SW1.13
- net 7P9: now also R2.2, SW1.15; no longer R1.2, SW1.16
- net 8P9: now also R1.2, SW1.16; no longer R2.2, SW1.15
- net +3V3 renamed +3.3VADC
- net GND renamed GND3
