File: mod. de exp. FPGA spartan 6 mimasV2 - copia/DISPLAY.kicad_sch (KiCad schematic)
At the start: 9 parts, among them U1 CA56-12CGKWA

Commit message: absolutamente todo
Parts:
- R17, R18, R19, R20, R21, R22, R23, R24: footprint Resistor_THT:R_Axial_DIN0207_L6.3mm_D2.5mm_P10.16mm_Horizontal -> Resistor_THT:R_Axial_DIN0207_L6.3mm_D2.5mm_P7.62mm_Horizontal
Connections:
- net 1P6: now also U1.6 (CA4); no longer U1.9 (CA2)
- net 1P7: now also R17.1; no longer R18.1
- net 2P6: now also U1.8 (CA3); no longer U1.12 (CA1)
- net 2P7: now also R18.1; no longer R17.1
- net 3P6: now also U1.9 (CA2); no longer U1.6 (CA4)
- net 3P7: now also R19.1; no longer R20.1
- net 4P6: now also U1.12 (CA1); no longer U1.8 (CA3)
- net 4P7: now also R20.1; no longer R19.1
- net 5P7: now also R21.1; no longer R22.1
- net 6P7: now also R22.1; no longer R21.1
- net 7P7: now also R23.1; no longer R24.1
- net 8P7: now also R24.1; no longer R23.1
