File: mod. de exp. FPGA spartan 6 mimasV2 - copia/LEDs.kicad_sch (KiCad schematic)
At the start: 16 parts

Commit message: absolutamente todo
Parts:
- R10, R11, R12, R13, R14, R15, R16, R9: footprint Resistor_THT:R_Axial_DIN0207_L6.3mm_D2.5mm_P10.16mm_Horizontal -> Resistor_THT:R_Axial_DIN0207_L6.3mm_D2.5mm_P7.62mm_Horizontal
Connections:
- net GND renamed GND2
