File: mod. de exp. FPGA spartan 6 mimasV2 - copia/PIN_HEADER_8X4.kicad_sch (KiCad schematic)
At the start: 4 parts, among them J1 P6, J2 P7, J3 P8, J4 P9

Commit message: absolutamente todo
Connections:
- net +3V3: no longer J2.1 (Pin_1), J2.2 (Pin_2), J3.1 (Pin_1), J3.2 (Pin_2), J4.1 (Pin_1), J4.2 (Pin_2)
- net GND: no longer J2.3 (Pin_3), J2.4 (Pin_4), J3.3 (Pin_3), J3.4 (Pin_4), J4.3 (Pin_3), J4.4 (Pin_4)
- new net +3.3V: J2.1 (Pin_1), J2.2 (Pin_2)
- new net +3.3VA: J3.1 (Pin_1), J3.2 (Pin_2)
- new net +3.3VADC: J4.1 (Pin_1), J4.2 (Pin_2)
- new net GND1: J2.3 (Pin_3), J2.4 (Pin_4)
- new net GND2: J3.3 (Pin_3), J3.4 (Pin_4)
- new net GND3: J4.3 (Pin_3), J4.4 (Pin_4)
