File: mod. de exp. FPGA spartan 6 mimasV2 - copia/PUSH.kicad_sch (KiCad schematic)
At the start: 8 parts, among them SW2 SW_Push, SW3 SW_Push, SW4 SW_Push, SW5 SW_Push

Commit message: absolutamente todo
Parts:
- R25, R26, R27, R28: footprint Resistor_THT:R_Axial_DIN0207_L6.3mm_D2.5mm_P10.16mm_Horizontal -> Resistor_THT:R_Axial_DIN0207_L6.3mm_D2.5mm_P7.62mm_Horizontal
Connections:
- net GND renamed GND2
