File: proyecto de cuatrinestre/CONTROL.kicad_sch (KiCad schematic)
At the start: 35 parts, among them IC1 MKE04Z128VLD4, J7 Screw_Terminal_01x06, J8 JTAG SWD CONNECTOR, SW1 SW_DIP_x08, SW2 SW_DIP_x04, SW3 SW_Push, Y1 8Mhz

Commit message: aja
Parts:
- removed R28, R29, R30, R31, R32, R33, R34, R35, R37, R38, R40, R41: 10k / 1%, Resistor_SMD:R_0805_2012Metric, symbol Device:R
- removed SW1: SW_DIP_x08, Button_Switch_THT:SW_DIP_SPSTx08_Slide_6.7x21.88mm_W7.62mm_P2.54mm_LowProfile, symbol Switch:SW_DIP_x08
- removed SW2: SW_DIP_x04, Button_Switch_THT:SW_DIP_SPSTx04_Slide_6.7x11.72mm_W7.62mm_P2.54mm_LowProfile, symbol Switch:SW_DIP_x04
- added U17: ESP32-WROOM-32, RF_Module:ESP32-WROOM-32, symbol RF_Module:ESP32-WROOM-32
Connections:
- new net: U17.1 (GND), U17.15 (GND), U17.38 (GND), U17.39 (GND)

Commit message: absolutamente todo
Parts:
- removed C14, C15, C16: 0.1uF / 50V, Capacitor_SMD:C_0805_2012Metric, symbol Device:C
- removed C6: 22pF / 50V, Capacitor_SMD:C_0805_2012Metric, symbol Device:C
- removed IC1: MKE04Z128VLD4, KiCad:QFP80P1200X1200X160-44N, symbol MKE04Z128VLD4:MKE04Z128VLD4
- removed J8: JTAG SWD CONNECTOR, Connector_PinHeader_2.54mm:PinHeader_2x03_P2.54mm_Vertical, symbol Connector:Screw_Terminal_01x06
- removed R36: 10k / 1%, Resistor_SMD:R_0805_2012Metric, symbol Device:R
- removed R49, R50, R51, R52, R53: 100K, Resistor_SMD:R_0805_2012Metric, symbol Device:R
- removed SW3: SW_Push, Button_Switch_THT:SW_PUSH_6mm, symbol Switch:SW_Push
- removed Y1: 8Mhz, Crystal:Crystal_SMD_HC49-SD, symbol Device:Crystal
- added J8: ESP32-JTAG, Connector_PinHeader_2.54mm:PinHeader_2x05_P2.54mm_Vertical, symbol nuevos simvolos:ESP32-JTAG
- added R28, R29, R30, R31, R32: 10K, Resistor_SMD:R_0805_2012Metric, symbol Device:R
- added R33: 22K, Resistor_SMD:R_0805_2012Metric, symbol Device:R
- C12: value 0.1uF / 50V -> 22uF
- C13: value 0.1uF / 50V -> 0.1uF
- C5: value 22pF / 50V -> 0.1uF
- R27: value 10k / 1% -> 22K
Connections:
- net +5V is gone; now on net VDD: C12.1, C13.1, J7.1 (Pin_1), R39.2
- net COM_RS485_LCD: now also U17.6 (IO34)
- net CON_RS485_eXT: now also U17.7 (IO35)
- net GND: now also U17.1 (GND), U17.15 (GND), U17.38 (GND), U17.39 (GND), J8.3 (GND), J8.9 (GNDDetect); no longer C5.1
- net INPUT_1_MICRO: now also U17.29 (IO5)
- net INPUT_2_MICRO: now also U17.26 (IO4)
- net INPUT_3_MICRO: now also U17.25 (IO0)
- net INPUT_4_MICRO: now also U17.24 (IO2)
- net RLY_FAN1_MICRO: now also U17.10 (IO25)
- net RLY_FAN2_MICRO: now also U17.11 (IO26)
- net RLY_FAN3_MICRO: now also U17.12 (IO27)
- net RLY_OUT1_MICRO: now also U17.36 (IO22)
- net RLY_OUT2_MICRO: now also U17.37 (IO23)
- net Rx_RS485_eXT: now also U17.34 (RXD0/IO3)
- net Rx_RS485_lcd: now also U17.27 (IO16)
- net Tx_RS485_LCD: now also U17.28 (IO17)
- net Tx_RS485_eXT: now also U17.35 (TXD0/IO1)
- net at D12.1 (K): now also U17.9 (IO33)
- net VDD: now reaches R27.2
- net VDD: now also C5.1, U17.2 (VDD), R28.2, R29.2, R30.2, R31.2, R32.2, R33.2; no longer C5.2
- net at R27.1: now also J8.1 (VTRef)
- net at J7.3 (Pin_3): now also U17.8 (IO32)
- net at J7.6 (Pin_6): now also U17.33 (IO21)
- net at J7.4 (Pin_4): now also U17.31 (IO19)
- net at J7.2 (Pin_2): now also U17.30 (IO18)
- net TMS: now reaches U17.13 (IO14)
- net TMS: now also J8.2 (TMS), R28.1
- net TDI: now reaches U17.14 (IO12)
- net TDI: now also J8.8 (TDI), R31.1
- net TCK: now reaches U17.16 (IO13)
- net TCK: now also J8.4 (TCK), R29.1
- net TDO: now reaches U17.23 (IO15)
- net TDO: now also J8.6 (TDO), R30.1
- net nRESET: now reaches U17.3 (EN)
- net nRESET: now also C5.2, J8.10 (nRESET), R32.1, R33.1
Other:
- moved on the sheet: C12, C13, D12, R39, U17
