File: proyecto de cuatrinestre/RELAY GROUP.kicad_sch (KiCad schematic)
At the start: 16 parts, among them U10 AZ921, U11 AZ921, U6 ULN2003A, U7 AZ921, U8 AZ921, U9 AZ921

Commit message: absolutamente todo
Connections:
- net CON-OUT1A: now also U7.3; no longer U7.4
- net CON-OUT1B: now also U7.4; no longer U7.3
- net CON-OUT2A: now also U8.3; no longer U8.4
- net CON-OUT2B: now also U8.4; no longer U8.3
- net at D9.1 (K), U6.12 (O5): now also U9.2; no longer U11.2
- net at D6.1 (K), U6.15 (O2): now also U7.2; no longer U8.2
- net at D5.1 (K), U6.16 (O1): now also U8.2; no longer U7.2
- net at D7.1 (K), U6.14 (O3): now also U11.2; no longer U9.2
Other:
- moved on the sheet: U7, U8
