File: proyecto de cuatrinestre/RS-485-EXTERNA.kicad_sch (KiCad schematic)
At the start: 11 parts, among them U1 TD521D485H-E, U12 SMBJ12CA

Commit message: absolutamente todo
Parts:
- removed R25, R26: 10, Resistor_SMD:R_0805_2012Metric, symbol Device:R
Connections:
- net at D11.2 (A2), R22.2, U1.9 (A)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: now also F2.1
- net at D11.1 (A1), R23.2, U1.8 (B)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: now also F1.1
- net +5V renamed VDD
