File: proyecto de cuatrinestre/RS-485-LCD.kicad_sch (KiCad schematic)
At the start: 8 parts, among them U13 SP485ECN-L, U14 SMBJ12CA

Commit message: absolutamente todo
Connections:
- net +5V renamed VDD
