File: proyecto de cuatrinestre/power suplay.kicad_sch (KiCad schematic)
At the start: 21 parts, among them J9 TP1X3, U15 LM7805_TO220, U16 B0505S-W2R2

Commit message: absolutamente todo
Parts:
- removed D15, D19: LED, LED_SMD:LED_0805_2012Metric, symbol Device:LED
- removed J9: TP1X3, Connector_PinHeader_2.54mm:PinHeader_1x03_P2.54mm_Vertical, symbol Connector:Screw_Terminal_01x03
- removed R46, R48: R, Resistor_SMD:R_0805_2012Metric, symbol Device:R
- removed U15: LM7805_TO220, Package_TO_SOT_THT:TO-220-3_Vertical, symbol Regulator_Linear:LM7805_TO220
- added U15: 3v3 NJM2885DL1-33, Package_TO_SOT_SMD:TO-252-2, symbol nuevos simvolos:3v3 NJM2885DL1-33
- F3: footprint Fuse:Fuseholder_Clip-5x20mm_Keystone_3517_Inline_P23.11x6.76mm_D1.70mm_Horizontal -> Fuse:Fuseholder_Cylinder-5x20mm_Schurter_0031_8201_Horizontal_Open
- U16: value B0505S-W2R2 -> B0303S-W2R2; footprint nuevo simbolo:B0505S-W2R2 -> B0505S-1WR2:CONV_B0505S-1WR2
Connections:
- net +5V is gone; now on net VDD: C10.1, C11.1, D17.1, R47.1, U16.2 (IN+)
- net +12V: now also U15.1 (Vin)
- net GND: now also U15.2 (GND)
- net VDD: now also U15.3 (Vout); no longer D18.1, U16.4 (OUT+)
- new net +3V3: D18.1, U16.4 (OUT+)
