File: proyecto de cuatrinestre/proyecto de cuatrinestre.kicad_sch (KiCad schematic)
At the start: 6 parts, among them J1 Screw_Terminal_01x02, J2 Screw_Terminal_01x02, J3 Screw_Terminal_01x02, J4 Screw_Terminal_01x03, J5 Screw_Terminal_01x08, J6 Screw_Terminal_01x08

Commit message: absolutamente todo
Connections:
- net ROOMLINK/CON-A-: now also J4.3 (Pin_3); no longer J4.2 (Pin_2)
- net ROOMLINK/CON-B+: now also J4.2 (Pin_2); no longer J4.3 (Pin_3)
