File: proyecto de cuatrinestre/proyecto de cuatrinestre.kicad_pcb (KiCad board)
At the start: 2 copper layers, 125 parts, among them IC1 MKE04Z128VLD4, J1 Screw_Terminal_01x02, J2 Screw_Terminal_01x02, J3 Screw_Terminal_01x02, J4 Screw_Terminal_01x03, J5 Screw_Terminal_01x08, J6 Screw_Terminal_01x08, J7 Screw_Terminal_01x06, J8 JTAG SWD CONNECTOR, J9 TP1X3, SW1 SW_DIP_x08, SW2 SW_DIP_x04, SW3 SW_Push, U1 TD521D485H-E, U10 AZ921, U11 AZ921, U12 SMBJ12CA, U13 SP485ECN-L, U14 SMBJ12CA, U15 LM7805_TO220, U16 B0505S-W2R2, U2 FODM2705, U3 FODM2705, U4 FODM2705, U5 FODM2705, U6 ULN2003A, U7 AZ921, U8 AZ921, U9 AZ921, Y1 8Mhz

Commit message: aja
Parts:
- added U17: ESP32-WROOM-32, RF_Module:ESP32-WROOM-32, F.Cu at (332.6, 183.2)
- moved C1 147.3 mm to (371.8, 115.3)
- moved C11 147.3 mm to (292.7, 80.4)
- moved C13 147.3 mm to (358.8, 44.6)
- moved C16 147.3 mm to (358.8, 47.6)
- moved C2 147.3 mm to (376.3, 108.6)
- moved C3 147.3 mm to (367.4, 118.3)
- moved C5 147.3 mm to (380.4, 28.3)
- moved C6 147.3 mm to (358.8, 41.6)
- moved C7 147.3 mm to (375.7, 65.6)
- moved C8 147.3 mm to (382.8, 60.1)
- moved D13 147.3 mm to (383.9, 54.7)
- moved D17 147.3 mm to (269.4, 101.3)
- moved D5 147.3 mm to (322.4, 93.7)
- moved D8 147.3 mm to (322.4, 90.6)
- moved F2 147.3 mm to (342.4, 100.9)
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Other:
- board outline added: 107 x 87.7 mm

Commit message: absolutamente todo
Parts:
- removed C14, C15, C16: 0.1uF / 50V, Capacitor_SMD:C_0805_2012Metric
- removed C6: 22pF / 50V, Capacitor_SMD:C_0805_2012Metric
- removed D15, D19: LED, LED_SMD:LED_0805_2012Metric
- removed IC1: MKE04Z128VLD4, KiCad:QFP80P1200X1200X160-44N
- removed J9: TP1X3, Connector_PinHeader_2.54mm:PinHeader_1x03_P2.54mm_Vertical
- removed R25, R26: 10, Resistor_SMD:R_0805_2012Metric
- removed R34, R35, R36, R37, R38, R40, R41: 10k / 1%, Resistor_SMD:R_0805_2012Metric
- removed R46, R48: R, Resistor_SMD:R_0805_2012Metric
- removed R49, R50, R51, R52, R53: 100K, Resistor_SMD:R_0805_2012Metric
- removed SW1: SW_DIP_x08, Button_Switch_THT:SW_DIP_SPSTx08_Slide_6.7x21.88mm_W7.62mm_P2.54mm_LowProfile
- removed SW2: SW_DIP_x04, Button_Switch_THT:SW_DIP_SPSTx04_Slide_6.7x11.72mm_W7.62mm_P2.54mm_LowProfile
- removed SW3: SW_Push, Button_Switch_THT:SW_PUSH_6mm
- removed Y1: 8Mhz, Crystal:Crystal_SMD_HC49-SD
- C12: value 0.1uF / 50V -> 22uF
- C13: value 0.1uF / 50V -> 0.1uF
- C5: value 22pF / 50V -> 0.1uF
- F3: footprint Fuse:Fuseholder_Clip-5x20mm_Keystone_3517_Inline_P23.11x6.76mm_D1.70mm_Horizontal -> Fuse:Fuseholder_Cylinder-5x20mm_Schurter_0031_8201_Horizontal_Open
- J8: value JTAG SWD CONNECTOR -> ESP32-JTAG; footprint Connector_PinHeader_2.54mm:PinHeader_2x03_P2.54mm_Vertical -> Connector_PinHeader_2.54mm:PinHeader_2x05_P2.54mm_Vertical
- R27, R33: value 10k / 1% -> 22K
- R28, R29, R30, R31, R32: value 10k / 1% -> 10K
- U15: value LM7805_TO220 -> 3v3 NJM2885DL1-33; footprint Package_TO_SOT_THT:TO-220-3_Vertical -> Package_TO_SOT_SMD:TO-252-2
- U16: value B0505S-W2R2 -> B0303S-W2R2; footprint nuevo simbolo:B0505S-W2R2 -> B0505S-1WR2:CONV_B0505S-1WR2
- moved R27 218.6 mm to (211.7, 142.1), turned to 90 degrees
- moved J8 217.5 mm to (204.0, 146.5)
- moved R29 215.4 mm to (211.7, 149.0), turned to 90 degrees
- moved R43 214.3 mm to (183.1, 114.8), turned to 90 degrees
- moved D13 213.0 mm to (179.4, 114.5), turned to 90 degrees
- moved R44 210.3 mm to (175.8, 114.8), turned to 90 degrees
- moved R30 207.0 mm to (211.7, 152.5), turned to 90 degrees
- moved U14 206.1 mm to (179.4, 119.8)
- moved R32 205.2 mm to (211.7, 159.4), turned to 90 degrees
- moved C8 201.3 mm to (191.2, 122.0), turned to 90 degrees
- moved R28 199.0 mm to (211.7, 145.6), turned to 90 degrees
- moved R31 196.3 mm to (211.7, 156.0), turned to 90 degrees
- moved C7 195.1 mm to (189.0, 122.0), turned to 90 degrees
- moved U13 192.8 mm to (196.2, 121.3), turned to 180 degrees
- moved J4 191.4 mm to (206.4, 188.5)
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Connections:
- C1 pad 1: Net-(C1-Pad1) -> /ROOMLINK/CONTROL/INPUT_1_MICRO
- C10 pad 1: +5V -> VDD
- C11 pad 1: +5V -> VDD
- C12 pad 1: +5V -> VDD
- C13 pad 1: +5V -> VDD
- C2 pad 1: Net-(C2-Pad1) -> /ROOMLINK/CONTROL/INPUT_2_MICRO
- C3 pad 1: Net-(C3-Pad1) -> /ROOMLINK/CONTROL/INPUT_4_MICRO
- C4 pad 1: Net-(C4-Pad1) -> /ROOMLINK/CONTROL/INPUT_3_MICRO
- C5 pad 1: GND -> VDD
- C5 pad 2: Net-(C5-Pad2) -> nRESET
- C7 pad 1: +5V -> VDD
- C8 pad 1: +5V -> VDD
- D11 pad 1: Net-(D11-Pad1) -> Net-(D11-A1)
- D11 pad 2: Net-(D11-Pad2) -> Net-(D11-A2)
- D12 pad 1: Net-(D12-Pad1) -> Net-(D12-K)
- D17 pad 1: +5V -> VDD
- D18 pad 1: VDD -> +3V3
- D5 pad 1: Net-(D5-Pad1) -> Net-(D5-K)
- D6 pad 1: Net-(D6-Pad1) -> Net-(D6-K)
- D7 pad 1: Net-(D7-Pad1) -> Net-(D7-K)
- D9 pad 1: Net-(D9-Pad1) -> Net-(D9-K)
- F1 pad 1: Net-(F1-Pad1) -> Net-(D11-A1)
- F2 pad 1: Net-(F2-Pad1) -> Net-(D11-A2)
- J4 pad 2: /ROOMLINK/CON-A- -> /ROOMLINK/CON-B+
- J4 pad 3: /ROOMLINK/CON-B+ -> /ROOMLINK/CON-A-
- J7 pad 1: +5V -> VDD
- J7 pad 2: Net-(IC1-Pad41) -> Net-(J7-Pin_2)
- J7 pad 3: Net-(IC1-Pad38) -> Net-(J7-Pin_3)
- J7 pad 4: Net-(IC1-Pad40) -> Net-(J7-Pin_4)
- J7 pad 6: Net-(IC1-Pad39) -> Net-(J7-Pin_6)
- J8 pad 1: Net-(IC1-Pad44) -> Net-(J8-VTRef)
- J8 pad 2: Net-(J8-Pad2) -> TMS
- J8 pad 3: Net-(IC1-Pad42) -> GND
- J8 pad 4: GND -> TCK
- J8 pad 5: Net-(C16-Pad1) -> unconnected-(J8-Pad5)
- J8 pad 6: Net-(J8-Pad6) -> TDO
- R1 pad 1: VDD -> +3V3
- R11 pad 1: VDD -> +3V3
- R13 pad 1: +5V -> VDD
- R14 pad 1: +5V -> VDD
- R15 pad 1: +5V -> VDD
- R16 pad 1: +5V -> VDD
- R22 pad 2: Net-(D11-Pad2) -> Net-(D11-A2)
- R23 pad 2: Net-(D11-Pad1) -> Net-(D11-A1)
- R27 pad 1: Net-(C6-Pad2) -> Net-(J8-VTRef)
- R27 pad 2: Net-(C5-Pad2) -> VDD
- R28 pad 1: Net-(IC1-Pad15) -> TMS
- R28 pad 2: +5V -> VDD
- R29 pad 1: Net-(IC1-Pad14) -> TCK
- R29 pad 2: +5V -> VDD
- R3 pad 1: VDD -> +3V3
- R30 pad 1: Net-(IC1-Pad12) -> TDO
- R30 pad 2: +5V -> VDD
- R31 pad 1: Net-(IC1-Pad11) -> TDI
- R31 pad 2: +5V -> VDD
- R32 pad 1: Net-(IC1-Pad4) -> nRESET
- R32 pad 2: +5V -> VDD
- R33 pad 1: Net-(IC1-Pad3) -> nRESET
- R33 pad 2: +5V -> VDD
- R39 pad 2: +5V -> VDD
- R47 pad 1: +5V -> VDD
- R5 pad 1: +5V -> VDD
- R6 pad 1: +5V -> VDD
- R7 pad 1: +5V -> VDD
- R8 pad 1: +5V -> VDD
- R9 pad 1: VDD -> +3V3
- U1 pad 1: +5V -> VDD
- U1 pad 8: Net-(D11-Pad1) -> Net-(D11-A1)
- U1 pad 9: Net-(D11-Pad2) -> Net-(D11-A2)
- U11 pad 2: Net-(D9-Pad1) -> Net-(D7-K)
- U12 pad 1: Net-(D11-Pad1) -> Net-(D11-A1)
- U12 pad 2: Net-(D11-Pad2) -> Net-(D11-A2)
- U13 pad 8: +5V -> VDD
- U15 pad 3: +5V -> VDD
- U16 pad 2: +5V -> VDD
- U16 pad 4: VDD -> +3V3
- U17 pad 1: Net-(U17-Pad1) -> GND
- U17 pad 10: unconnected-(U17-Pad10) -> /ROOMLINK/CONTROL/RLY_FAN1_MICRO
- U17 pad 11: unconnected-(U17-Pad11) -> /ROOMLINK/CONTROL/RLY_FAN2_MICRO
- U17 pad 12: unconnected-(U17-Pad12) -> /ROOMLINK/CONTROL/RLY_FAN3_MICRO
- U17 pad 13: unconnected-(U17-Pad13) -> TMS
- U17 pad 14: unconnected-(U17-Pad14) -> TDI
- U17 pad 15: Net-(U17-Pad1) -> GND
- U17 pad 16: unconnected-(U17-Pad16) -> TCK
- U17 pad 2: unconnected-(U17-Pad2) -> VDD
- U17 pad 23: unconnected-(U17-Pad23) -> TDO
- U17 pad 24: unconnected-(U17-Pad24) -> /ROOMLINK/CONTROL/INPUT_4_MICRO
- U17 pad 25: unconnected-(U17-Pad25) -> /ROOMLINK/CONTROL/INPUT_3_MICRO
- U17 pad 26: unconnected-(U17-Pad26) -> /ROOMLINK/CONTROL/INPUT_2_MICRO
- U17 pad 27: unconnected-(U17-Pad27) -> /ROOMLINK/CONTROL/Rx_RS485_lcd
- U17 pad 28: unconnected-(U17-Pad28) -> /ROOMLINK/CONTROL/Tx_RS485_LCD
- U17 pad 29: unconnected-(U17-Pad29) -> /ROOMLINK/CONTROL/INPUT_1_MICRO
- U17 pad 3: unconnected-(U17-Pad3) -> nRESET
- U17 pad 30: unconnected-(U17-Pad30) -> Net-(J7-Pin_2)
- U17 pad 31: unconnected-(U17-Pad31) -> Net-(J7-Pin_4)
- U17 pad 33: unconnected-(U17-Pad33) -> Net-(J7-Pin_6)
- U17 pad 34: unconnected-(U17-Pad34) -> /ROOMLINK/CONTROL/Rx_RS485_eXT
- U17 pad 35: unconnected-(U17-Pad35) -> /ROOMLINK/CONTROL/Tx_RS485_eXT
- U17 pad 36: unconnected-(U17-Pad36) -> /ROOMLINK/CONTROL/RLY_OUT1_MICRO
- U17 pad 37: unconnected-(U17-Pad37) -> /ROOMLINK/CONTROL/RLY_OUT2_MICRO
- U17 pad 38: Net-(U17-Pad1) -> GND
- U17 pad 39: Net-(U17-Pad1) -> GND
- U17 pad 6: unconnected-(U17-Pad6) -> /ROOMLINK/CONTROL/COM_RS485_LCD
- U17 pad 7: unconnected-(U17-Pad7) -> /ROOMLINK/CONTROL/CON_RS485_eXT
- U17 pad 8: unconnected-(U17-Pad8) -> Net-(J7-Pin_3)
- U17 pad 9: unconnected-(U17-Pad9) -> Net-(D12-K)
- U2 pad 4: Net-(C1-Pad1) -> /ROOMLINK/CONTROL/INPUT_1_MICRO
- U3 pad 4: Net-(C2-Pad1) -> /ROOMLINK/CONTROL/INPUT_2_MICRO
- U4 pad 4: Net-(C3-Pad1) -> /ROOMLINK/CONTROL/INPUT_4_MICRO
- U5 pad 4: Net-(C4-Pad1) -> /ROOMLINK/CONTROL/INPUT_3_MICRO
- U6 pad 12: Net-(D9-Pad1) -> Net-(D9-K)
- U6 pad 14: Net-(D7-Pad1) -> Net-(D7-K)
- U6 pad 15: Net-(D6-Pad1) -> Net-(D6-K)
- U6 pad 16: Net-(D5-Pad1) -> Net-(D5-K)
- U7 pad 2: Net-(D5-Pad1) -> Net-(D6-K)
- U7 pad 3: /ROOMLINK/CON-OUT1B -> /ROOMLINK/CON-OUT1A
- U7 pad 4: /ROOMLINK/CON-OUT1A -> /ROOMLINK/CON-OUT1B
- U8 pad 2: Net-(D6-Pad1) -> Net-(D5-K)
- U8 pad 3: /ROOMLINK/CON-OUT2B -> /ROOMLINK/CON-OUT2A
- U8 pad 4: /ROOMLINK/CON-OUT2A -> /ROOMLINK/CON-OUT2B
- U9 pad 2: Net-(D7-Pad1) -> Net-(D9-K)
Routing:
- net +12V: track 0.00 -> 113.2 mm, vias 0 -> 8
- net /ROOMLINK/CONTROL/RLY_OUT1_MICRO: track 0.00 -> 92.6 mm, vias 0 -> 2
- net /ROOMLINK/CONTROL/RLY_OUT2_MICRO: track 0.00 -> 89.0 mm, vias 0 -> 2
- net /ROOMLINK/CONTROL/Rx_RS485_lcd: track 0.00 -> 84.2 mm, vias 0 -> 2
- net /ROOMLINK/CONTROL/Tx_RS485_LCD: track 0.00 -> 82.1 mm, vias 0 -> 2
- net /ROOMLINK/CONTROL/Tx_RS485_eXT: track 0.00 -> 65.8 mm
- net nRESET: track 0.00 -> 62.7 mm, vias 0 -> 2
- net /ROOMLINK/CONTROL/COM_RS485_LCD: track 0.00 -> 61.7 mm, vias 0 -> 2
- net GND: track 0.00 -> 60.8 mm, vias 0 -> 20
- net /ROOMLINK/CONTROL/CON_RS485_eXT: track 0.00 -> 57.6 mm, vias 0 -> 2
- net /ROOMLINK/CONTROL/Rx_RS485_eXT: track 0.00 -> 54.1 mm
- net /ROOMLINK/CONTROL/RLY_FAN3_MICRO: track 0.00 -> 51.7 mm, vias 0 -> 2
- net /ROOMLINK/CONTROL/RLY_FAN2_MICRO: track 0.00 -> 50.9 mm
- net Net-(D5-K): track 0.00 -> 49.1 mm, vias 0 -> 2
- net /ROOMLINK/CON-DC+: track 0.00 -> 47.3 mm, vias 0 -> 1
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- added copper zone on In1.Cu, net GND
- added copper zone on B.Cu, net GNDA
- added copper zone on In2.Cu, net VDD
Other:
- board size 107 x 87.7 mm -> 102.4 x 83.1 mm
- copper layers 2 -> 4

Commit message: ULTIMA ACTUALIZACION
Routing:
- net /ROOMLINK/CON-DC-: track 42.2 -> 40.8 mm
Changed lines of the file:
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@@
   (segment (start 261.68 177.4875) (end 259.2 177.4875) (width 0.5) (layer "F.Cu") (net 31))
   (segment (start 259.2 177.4875) (end 259.175 177.5125) (width 0.5) (layer "F.Cu") (net 31))
-  (segment (start 165.03 133.026) (end 171.196 139.192) (width 0.8) (layer "F.Cu") (net 32))
+  (segment (start 176.215 135.75) (end 178 137.535) (width 0.8) (layer "F.Cu") (net 32))
   (segment (start 181.069166 137.535) (end 178 137.535) (width 0.8) (layer "F.Cu") (net 32))
-  (segment (start 176.343 139.192) (end 178 137.535) (width 0.8) (layer "F.Cu") (net 32))
+  (segment (start 165.03 133.026) (end 167.754 135.75) (width 0.8) (layer "F.Cu") (net 32))
   (segment (start 165.03 110.0875) (end 165.03 133.026) (width 0.8) (layer "F.Cu") (net 32))
-  (segment (start 171.196 139.192) (end 176.343 139.192) (width 0.8) (layer "F.Cu") (net 32))
+  (segment (start 167.754 135.75) (end 176.215 135.75) (width 0.8) (layer "F.Cu") (net 32))
   (segment (start 187.75 172.4) (end 186.9 171.55) (width 2) (layer "B.Cu") (net 33))
   (segment (start 168.71 147.1) (end 168.71 149.406) (width 2) (layer "B.Cu") (net 33))

Commit message: terminacion
Parts:
- moved F4 31.6 mm to (170.2, 115.0), turned to 90 degrees
- moved R45 26.4 mm to (167.2, 120.0)
- moved D14 25.3 mm to (163.8, 120.0)
- moved F5 25.3 mm to (165.0, 115.0), turned to 90 degrees
Routing:
- net /ROOMLINK/CON-DC+: track 47.3 -> 11.4 mm, vias 1 -> 0
- net +12V: track 113.2 -> 146.9 mm, vias 8 -> 6
- net /ROOMLINK/CON-DC-: track 40.8 -> 11.5 mm
- net Net-(D5-K): track 49.1 -> 51.2 mm
- net Net-(D14-A): track 3.08 -> 1.65 mm
Other:
- outline, holes or cut-outs redrawn
