File: proyecto final/fuente.kicad_sch (KiCad schematic)
At the start: 18 parts, among them U1 fuse_CC12H1.5A-TR, U2 3v3 NJM2885DL1-33, U3 LM7805_TO220, U4 fuse_CC12H1.5A-TR, U5 fuse_CC12H1.5A-TR

Commit message: absolutamente todo
Parts:
- added C7, C8: 100uF / 25V, Capacitor_THT:CP_Radial_D6.3mm_P2.50mm, symbol Device:C_Polarized
Connections:
- net +12V: now also C7.1, C8.1
- net GND: now also C7.2, C8.2
Other:
- moved on the sheet: C2, C4, D3, R5, U3, U5
