File: proyecto final/micro.kicad_sch (KiCad schematic)
At the start: 3 parts, among them J3 IO_IZQUIERDA, J4 IO_DERECHA, SW1 SW_DIP_x01

Commit message: CAMBIO DE HEADER
Parts:
- J3, J4: footprint Connector_PinHeader_2.54mm:PinHeader_1x17_P2.54mm_Vertical -> Connector_PinSocket_2.54mm:PinSocket_1x17_P2.54mm_Vertical
Changed lines of the file:
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@@
     (property "Reference" "J4" (id 0) (at 165.1508 74.295 0))
     (property "Value" "IO_DERECHA" (id 1) (at 165.1508 76.835 0))
-    (property "Footprint" "Connector_PinHeader_2.54mm:PinHeader_1x17_P2.54mm_Vertical" (id 2) (at 165.7096 100.1522 0)
+    (property "Footprint" "Connector_PinSocket_2.54mm:PinSocket_1x17_P2.54mm_Vertical" (id 2) (at 165.7096 100.1522 0)
       (effects (font (size 1.27 1.27)) hide)
     )
@@
       (effects (font (size 1.27 1.27)) (justify left))
     )
-    (property "Footprint" "Connector_PinHeader_2.54mm:PinHeader_1x17_P2.54mm_Vertical" (id 2) (at 135.9916 100.1522 0)
+    (property "Footprint" "Connector_PinSocket_2.54mm:PinSocket_1x17_P2.54mm_Vertical" (id 2) (at 135.9916 100.1522 0)
       (effects (font (size 1.27 1.27)) hide)
     )

Commit message: absolutamente todo
Parts:
- added SW2: 3V3, Connector_PinHeader_2.54mm:PinHeader_1x02_P2.54mm_Vertical, symbol Switch:SW_DIP_x01
- SW1: value SW_DIP_x01 -> 5V; footprint Button_Switch_THT:SW_DIP_SPSTx01_Slide_9.78x4.72mm_W7.62mm_P2.54mm -> Connector_PinHeader_2.54mm:PinHeader_1x02_P2.54mm_Vertical
Connections:
- net +3V3: now also SW2.1; no longer SW1.1
- net +5VA: now also SW1.2
- net at J3.2 (Pin_2): now also SW2.2; no longer SW1.2
- new net +5V: SW1.1
