File: proyecto final/proyecto final.kicad_pcb (KiCad board)
At the start: 4 copper layers, 68.2 x 89.7 mm, 42 parts, among them J1 AC input, J10 5V, J11 12V, J12 12V, J13 inonizador input, J14 inonizador input, J15 GND, J16 GND, J2 inonizador input, J3 IO_IZQUIERDA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

Commit message: CAMBIO DE HEADER
Parts:
- J3, J4: footprint Connector_PinHeader_2.54mm:PinHeader_1x17_P2.54mm_Vertical -> Connector_PinSocket_2.54mm:PinSocket_1x17_P2.54mm_Vertical
Changed lines of the file:
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@@
     )
   )
-  (footprint "Connector_PinHeader_2.54mm:PinHeader_1x17_P2.54mm_Vertical" locked (layer "F.Cu")
+  (footprint "Connector_PinSocket_2.54mm:PinSocket_1x17_P2.54mm_Vertical" locked (layer "F.Cu")
     (at 130 96.78)
-    (descr "Through hole straight pin header, 1x17, 2.54mm pitch, single row")
-    (tags "Through hole pin header THT 1x17 2.54mm single row")
+    (descr "Through hole straight socket strip, 1x17, 2.54mm pitch, single row (from Kicad 4.0.7), script generated")
+    (tags "Through hole socket strip THT 1x17 2.54mm single row")
     (property "Sheetfile" "Archivo: micro.kicad_sch")
     (property "Sheetname" "micro")
     (attr through_hole)
-    (fp_text reference "J3" (at -0.01 -2.4) (layer "F.SilkS") hide
-      (effects (font (size 1 1) (thickness 0.15)))
-    )
-    (fp_text value "IO_IZQUIERDA" (at 0 42.97) (layer "F.Fab") hide
-      (effects (font (size 1 1) (thickness 0.15)))
-    )
-    (fp_text user "${REFERENCE}" (at 0 20.32 90) (layer "F.Fab") hide
-      (effects (font (size 1 1) (thickness 0.15)))
-    )
+    (fp_text reference "J3" (at 0 -2.77) (layer "F.SilkS")
+      (effects (font (size 1 1) (thickness 0.15)))
+    )
+    (fp_text value "IO_IZQUIERDA" (at 0 43.41) (layer "F.Fab")
+      (effects (font (size 1 1) (thickness 0.15)))
+    )
+    (fp_text user "${REFERENCE}" (at 0 20.32 90) (layer "F.Fab")
+      (effects (font (size 1 1) (thickness 0.15)))
+    )
+    (fp_line (start 0 -1.33) (end 1.33 -1.33) (layer "F.SilkS") (width 0.12))
+    (fp_line (start -1.33 41.97) (end 1.33 41.97) (layer "F.SilkS") (width 0.12))
+    (fp_line (start -1.33 1.27) (end -1.33 41.97) (layer "F.SilkS") (width 0.12))
+    (fp_line (start 1.33 -1.33) (end 1.33 0) (layer "F.SilkS") (width 0.12))
     (fp_line (start 1.33 1.27) (end 1.33 41.97) (layer "F.SilkS") (width 0.12))
-    (fp_line (start -1.33 41.97) (end 1.33 41.97) (layer "F.SilkS") (width 0.12))
     (fp_line (start -1.33 1.27) (end 1.33 1.27) (layer "F.SilkS") (width 0.12))
-    (fp_line (start -1.33 1.27) (end -1.33 41.97) (layer "F.SilkS") (width 0.12))
-    (fp_line (start -1.33 0) (end -1.33 -1.33) (layer "F.SilkS") (width 0.12))
-    (fp_line (start -1.33 -1.33) (end 0 -1.33) (layer "F.SilkS") (width 0.12))
-    (fp_line (start 1.8 42.45) (end 1.8 -1.8) (layer "F.CrtYd") (width 0.05))
-    (fp_line (start -1.8 -1.8) (end -1.8 42.45) (layer "F.CrtYd") (width 0.05))
-    (fp_line (start -1.8 42.45) (end 1.8 42.45) (layer "F.CrtYd") (width 0.05))
-    (fp_line (start 1.8 -1.8) (end -1.8 -1.8) (layer "F.CrtYd") (width 0.05))
-    (fp_line (start -1.27 41.91) (end -1.27 -0.635) (layer "F.Fab") (width 0.1))
+    (fp_line (start 1.75 -1.8) (end 1.75 42.4) (layer "F.CrtYd") (width 0.05))
+    (fp_line (start -1.8 42.4) (end -1.8 -1.8) (layer "F.CrtYd") (width 0.05))
+    (fp_line (start 1.75 42.4) (end -1.8 42.4) (layer "F.CrtYd") (width 0.05))
+    (fp_line (start -1.8 -1.8) (end 1.75 -1.8) (layer "F.CrtYd") (width 0.05))
+    (fp_line (start -1.27 -1.27) (end 0.635 -1.27) (layer "F.Fab") (width 0.1))
+    (fp_line (start -1.27 41.91) (end -1.27 -1.27) (layer "F.Fab") (width 0.1))
     (fp_line (start 1.27 41.91) (end -1.27 41.91) (layer "F.Fab") (width 0.1))
-    (fp_line (start 1.27 -1.27) (end 1.27 41.91) (layer "F.Fab") (width 0.1))
-    (fp_line (start -0.635 -1.27) (end 1.27 -1.27) (layer "F.Fab") (width 0.1))
-    (fp_line (start -1.27 -0.635) (end -0.635 -1.27) (layer "F.Fab") (width 0.1))
+    (fp_line (start 1.27 -0.635) (end 1.27 41.91) (layer "F.Fab") (width 0.1))
+    (fp_line (start 0.635 -1.27) (end 1.27 -0.635) (layer "F.Fab") (width 0.1))
     (pad "1" thru_hole rect locked (at 0 0) (size 1.7 1.7) (drill 1) (layers *.Cu *.Mask)
       (net 2 "GND") (pinfunction "Pin_1") (pintype "passive"))
@@
     (pad "17" thru_hole oval locked (at 0 40.64) (size 1.7 1.7) (drill 1) (layers *.Cu *.Mask)
       (net 2 "GND") (pinfunction "Pin_17") (pintype "passive"))
-    (model "${KICAD6_3DMODEL_DIR}/Connector_PinHeader_2.54mm.3dshapes/PinHeader_1x17_P2.54mm_Vertical.wrl"
+    (model "${KICAD6_3DMODEL_DIR}/Connector_PinSocket_2.54mm.3dshapes/PinSocket_1x17_P2.54mm_Vertical.wrl"
       (offset (xyz 0 0 0))
       (scale (xyz 1 1 1))
@@
     )
   )
-  (footprint "Connector_PinHeader_2.54mm:PinHeader_1x17_P2.54mm_Vertical" locked (layer "F.Cu")
+  (footprint "Connector_PinSocket_2.54mm:PinSocket_1x17_P2.54mm_Vertical" locked (layer "F.Cu")
     (at 150.86 96.78)
-    (descr "Through hole straight pin header, 1x17, 2.54mm pitch, single row")
-    (tags "Through hole pin header THT 1x17 2.54mm single row")
+    (descr "Through hole straight socket strip, 1x17, 2.54mm pitch, single row (from Kicad 4.0.7), script generated")
+    (tags "Through hole socket strip THT 1x17 2.54mm single row")
     (property "Sheetfile" "Archivo: micro.kicad_sch")
     (property "Sheetname" "micro")
     (attr through_hole)
-    (fp_text reference "J4" (at 0 -2.33) (layer "F.SilkS") hide
-      (effects (font (size 1 1) (thickness 0.15)))
-    )
-    (fp_text value "IO_DERECHA" (at 0 42.97) (layer "F.Fab") hide
-      (effects (font (size 1 1) (thickness 0.15)))
-    )
-    (fp_text user "${REFERENCE}" (at 0 20.32 90) (layer "F.Fab") hide
-      (effects (font (size 1 1) (thickness 0.15)))
-    )
+    (fp_text reference "J4" (at 0 -2.77) (layer "F.SilkS")
+      (effects (font (size 1 1) (thickness 0.15)))
+    )
+    (fp_text value "IO_DERECHA" (at 0 43.41) (layer "F.Fab")
+      (effects (font (size 1 1) (thickness 0.15)))
+    )
+    (fp_text user "${REFERENCE}" (at 0 20.32 90) (layer "F.Fab")
+      (effects (font (size 1 1) (thickness 0.15)))
+    )
+    (fp_line (start -1.33 1.27) (end 1.33 1.27) (layer "F.SilkS") (width 0.12))
     (fp_line (start -1.33 41.97) (end 1.33 41.97) (layer "F.SilkS") (width 0.12))
     (fp_line (start -1.33 1.27) (end -1.33 41.97) (layer "F.SilkS") (width 0.12))
-    (fp_line (start -1.33 1.27) (end 1.33 1.27) (layer "F.SilkS") (width 0.12))
-    (fp_line (start -1.33 0) (end -1.33 -1.33) (layer "F.SilkS") (width 0.12))
-    (fp_line (start -1.33 -1.33) (end 0 -1.33) (layer "F.SilkS") (width 0.12))
+    (fp_line (start 0 -1.33) (end 1.33 -1.33) (layer "F.SilkS") (width 0.12))
     (fp_line (start 1.33 1.27) (end 1.33 41.97) (layer "F.SilkS") (width 0.12))
-    (fp_line (start 1.8 -1.8) (end -1.8 -1.8) (layer "F.CrtYd") (width 0.05))
-    (fp_line (start -1.8 42.45) (end 1.8 42.45) (layer "F.CrtYd") (width 0.05))
-    (fp_line (start -1.8 -1.8) (end -1.8 42.45) (layer "F.CrtYd") (width 0.05))
-    (fp_line (start 1.8 42.45) (end 1.8 -1.8) (layer "F.CrtYd") (width 0.05))
+    (fp_line (start 1.33 -1.33) (end 1.33 0) (layer "F.SilkS") (width 0.12))
+    (fp_line (start -1.8 42.4) (end -1.8 -1.8) (layer "F.CrtYd") (width 0.05))
+    (fp_line (start 1.75 42.4) (end -1.8 42.4) (layer "F.CrtYd") (width 0.05))
+    (fp_line (start -1.8 -1.8) (end 1.75 -1.8) (layer "F.CrtYd") (width 0.05))
+    (fp_line (start 1.75 -1.8) (end 1.75 42.4) (layer "F.CrtYd") (width 0.05))
     (fp_line (start 1.27 41.91) (end -1.27 41.91) (layer "F.Fab") (width 0.1))
-    (fp_line (start -0.635 -1.27) (end 1.27 -1.27) (layer "F.Fab") (width 0.1))
-    (fp_line (start 1.27 -1.27) (end 1.27 41.91) (layer "F.Fab") (width 0.1))
-    (fp_line (start -1.27 -0.635) (end -0.635 -1.27) (layer "F.Fab") (width 0.1))
-    (fp_line (start -1.27 41.91) (end -1.27 -0.635) (layer "F.Fab") (width 0.1))
+    (fp_line (start -1.27 -1.27) (end 0.635 -1.27) (layer "F.Fab") (width 0.1))
+    (fp_line (start -1.27 41.91) (end -1.27 -1.27) (layer "F.Fab") (width 0.1))
+    (fp_line (start 0.635 -1.27) (end 1.27 -0.635) (layer "F.Fab") (width 0.1))
+    (fp_line (start 1.27 -0.635) (end 1.27 41.91) (layer "F.Fab") (width 0.1))
     (pad "1" thru_hole rect locked (at 0 0) (size 1.7 1.7) (drill 1) (layers *.Cu *.Mask)
       (net 2 "GND") (pinfunction "Pin_1") (pintype "passive"))
@@
     (pad "17" thru_hole oval locked (at 0 40.64) (size 1.7 1.7) (drill 1) (layers *.Cu *.Mask)
       (net 41 "/header2/12") (pinfunction "Pin_17") (pintype "passive"))
-    (model "${KICAD6_3DMODEL_DIR}/Connector_PinHeader_2.54mm.3dshapes/PinHeader_1x17_P2.54mm_Vertical.wrl"
-      (offset (xyz 0 0 0))
-      (scale (xyz 1 1 1))
+    (model "${KICAD6_3DMODEL_DIR}/Connector_PinSocket_2.54mm.3dshapes/PinSocket_1x17_P2.54mm_Vertical.wrl"
+      (offset (xyz 0 0 0))
+      (scale (xyz 1 1 1))

Commit message: absolutamente todo
Parts:
- added C7: 100uF / 25V, Capacitor_THT:CP_Radial_D6.3mm_P2.50mm, F.Cu at (129.1, 84.0)
- added C8: 100uF / 25V, Capacitor_THT:CP_Radial_D6.3mm_P2.50mm, F.Cu at (161.1, 54.5)
- added SW2: 3V3, Connector_PinHeader_2.54mm:PinHeader_1x02_P2.54mm_Vertical, F.Cu at (162.3, 88.3)
- SW1: value SW_DIP_x01 -> 5V; footprint Button_Switch_THT:SW_DIP_SPSTx01_Slide_9.78x4.72mm_W7.62mm_P2.54mm -> Connector_PinHeader_2.54mm:PinHeader_1x02_P2.54mm_Vertical
- moved SW1 6.21 mm to (159.7, 92.0), turned to 90 degrees
Connections:
- SW1 pad 1: +3V3 -> +5V
- SW1 pad 2: Net-(J3-Pad2) -> +5VA
Routing:
- net +5VA: track 0.00 -> 66.1 mm
- net +12V: track 110.5 -> 151.2 mm, vias 0 -> 1
- net +5V: track 123.4 -> 148.8 mm
- net Net-(F1-Pad1): track 25.6 -> 45.9 mm
- net Net-(J3-Pad2): track 31.7 -> 34.3 mm
- net +3V3: track 17.9 -> 20.4 mm
- net /proyecto_final/amperimetro/36: track 23.3 -> 23.9 mm
- added copper zone on B.Cu, net GND
- removed copper zone on In2.Cu, net +12V
- removed copper zone on B.Cu, net +5V
- removed copper zone on In1.Cu, net GND
Other:
- copper layers 4 -> 2
